File: cad/_autosave-RPi_Zero_pHat_Template.kicad_sch (KiCad schematic)
At the start: 88 parts, among them J101 Conn_01x03, J102 Conn_01x03, J103 Conn_01x03, J104 Conn_01x03, J105 Conn_01x03, J106 Conn_01x03, J107 Conn_01x03, J108 Conn_02x05_Odd_Even, J109 Conn_01x02, J110 Conn_01x02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

Commit message: add led
Parts:
- renumbered R135 to R132, R132 to R133, R133 to R134, R134 to R135
Connections:
- net LED: now also J115.18 (GPIO24)
