File: cad/MoBoControl.kicad_sch (KiCad schematic)
At the start: 88 parts, among them J101 Conn_01x03, J102 Conn_01x03, J103 Conn_01x03, J104 Conn_01x03, J105 Conn_01x03, J106 Conn_01x03, J107 Conn_01x03, J108 Conn_02x05_Odd_Even, J109 Conn_01x02, J110 Conn_01x02, J111 Conn_01x04, J112 USB_A, J113 Conn_02x05_Odd_Even, J114 power_input, J115 RPi_GPIO, J116 Conn_02x10_Odd_Even, U1 MCP23017, U101 ASSR-1218, U102 ASSR-1218, U103 ASSR-1218, U104 ASSR-1218, U105 ASSR-1218, U106 ASSR-1218, U107 ASSR-1218, U108 ASSR-1218, U109 ASSR-1218, U110 ASSR-1218, U111 ASSR-1218, U112 ASSR-1218, U113 ASSR-1218, U114 ASSR-1218, U115 ASSR-1218, U116 ASSR-1218

Commit message: rev1 cleanup
Parts:
- renumbered R135 to R132, R132 to R133, R133 to R134, R134 to R135
Connections:
- net GND: now also J114.2 (Pin_2)
- net LED: now also J115.18 (GPIO24)
Other:
- note added: "DEBUG LED"
- note added: "JUMPERS"
- note added: "PI HEADER"
- note added: "USB"
- note added: "VARIOUS PORTS"
- title: (none) -> MoBoControl Board
- moved on the sheet: C101, C102, D101, D102, D103, D104, D105, D106, D107, D108, D109, D110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

Commit message: Mobo V2 sent off for production
Parts:
- removed J109: Conn_01x02, Connector_PinHeader_2.54mm:PinHeader_1x02_P2.54mm_Vertical, symbol Connector_Generic:Conn_01x02
- added C103: 22uF, Capacitor_SMD:C_0805_2012Metric, symbol Device:CP_Small
- added C104, C105, C106, C107, C108: .1uF, Capacitor_SMD:C_0603_1608Metric, symbol Device:C_Small
- added H101, H102, H103, H104: MountingHole, MountingHole:MountingHole_3.2mm_M3_DIN965, symbol Mechanical:MountingHole
- added J105: Conn_02x04_Odd_Even, Connector_PinHeader_2.54mm:PinHeader_2x04_P2.54mm_Vertical, symbol Connector_Generic:Conn_02x04_Odd_Even
- added J112: Conn_02x03_Odd_Even, Connector_PinHeader_2.54mm:PinHeader_2x03_P2.54mm_Vertical, symbol Connector_Generic:Conn_02x03_Odd_Even
- added J117, J118: Conn_01x15, Connector_PinSocket_2.54mm:PinSocket_1x15_P2.54mm_Vertical, symbol Connector_Generic:Conn_01x15
- added R134, R135, R136, R137, R138, R139, R140, R141: 4.7k, Resistor_SMD:R_0603_1608Metric, symbol Device:R_Small
- added SW101, SW102: SW_Push, Button_Switch_SMD:SWITCH_2x3_SMD_TACTILE_GREEN, symbol Switch:SW_Push
- added U118: MAX232, Package_SO:SOIC-16_3.9x9.9mm_P1.27mm, symbol Interface_UART:MAX232
- renumbered D103 to D101, D104 to D102, D105 to D103, D106 to D104, D101 to D105, D102 to D106, D113 to D109, D114 to D110, D109 to D113, D110 to D114, J102 to J101, J103 to J102, J101 to J103, J107 to J106, J106 to J107, J105 to J108, J114 to J109, J112 to J111, J111 to J113, J113 to J114, J108 to J119, R103 to R101, R104 to R102, R105 to R103, R106 to R104, R101 to R105, R102 to R106, R111 to R109, R112 to R110, R113 to R111, R114 to R112, R109 to R113, R110 to R114, R129 to R117, R121 to R118, R122 to R119, R130 to R120, R119 to R121, R120 to R122, R117 to R123, R118 to R124, R127 to R125, R128 to R126, R125 to R127, R126 to R128, R123 to R129, R124 to R130, R134 to R131, R135 to R132, R132 to R133, R131 to R142, R133 to R143, U103 to U101, U104 to U102, U105 to U103, U106 to U104, U101 to U105, U102 to U106, U115 to U109, U113 to U110, U114 to U111, U116 to U112, U111 to U113, U112 to U114, U109 to U115, U110 to U116
Connections:
- net +3V3: now also C103.1, C106.1, J118.15 (Pin_15), U118.16 (VCC); no longer J115.17 (3.3V)
- net +5V: now also J117.15 (Pin_15)
- net GND: now also J110.2 (Pin_2), C103.2, C106.2, C108.2, J112.2 (Pin_2), J112.4 (Pin_4), J112.6 (Pin_6), J117.14 (Pin_14), J118.14 (Pin_14), R135.2, R137.2, R139.2, R141.2, U118.15 (GND)
- net RX: now also U118.14 (T1OUT); no longer J115.10 (GPIO15_RXD0)
- net TX: now also U118.13 (R1IN); no longer J115.8 (GPIO14_TXD0)
- net D34: now reaches J115.27 (ID_SD)
- net D34: now also J117.4 (Pin_4), R136.2, R137.1
- net D39: now reaches J115.31 (GPIO06)
- net D39: now also J117.3 (Pin_3), R138.2, R139.1
- net D36: now reaches J115.36 (GPIO16)
- net D36: now also J117.2 (Pin_2), R140.2, R141.1
- net D12: now reaches J115.7 (GPIO04_GCLK)
- net D12: now also J117.12 (Pin_12), R134.2, R135.1
- net at U109.4: now also J105.6 (Pin_6), J105.8 (Pin_8), SW101.1
- net at U109.3: now also J105.5 (Pin_5), J105.7 (Pin_7), SW101.2
- net at U112.3: now also J105.2 (Pin_2), J105.4 (Pin_4), SW102.1; no longer J110.2 (Pin_2)
- net at U112.4: now also J105.1 (Pin_1), J105.3 (Pin_3), SW102.2; no longer J110.1 (Pin_1)
- net IO_SCL renamed D27
- net D27: now also J117.10 (Pin_10)
- net IO_SDA renamed D26
- net D26: now also J117.9 (Pin_9)
- net LAD0 renamed D19
- net D19: now also J118.6 (Pin_6)
- net LAD1 renamed D23
- net D23: now also J118.1 (Pin_1)
- net LAD2 renamed D15
- net D15: now also J118.13 (Pin_13)
- net LAD3 renamed D32
- net D32: now also J117.6 (Pin_6)
- net LCLK renamed D18
- net D18: now also J118.7 (Pin_7)
- net LDRQ renamed D21
- net D21: now also J118.5 (Pin_5)
- net LED renamed D2
- net D2: now also J118.12 (Pin_12)
- net LFRAME renamed D25
- net D25: now also J117.8 (Pin_8)
- net LPCPD renamed D22
- net D22: now also J118.2 (Pin_2)
- net LRESET renamed D33
- net D33: now also J117.7 (Pin_7)
- net SCL renamed D16
- net D16: now also J118.10 (Pin_10)
- net SDA renamed D4
- net D4: now also J118.11 (Pin_11)
- net SER_IRQ renamed D5
- net D5: now also J118.8 (Pin_8)
- net SMB_CLK renamed D14
- net D14: now also J117.11 (Pin_11)
- net SMB_DAT renamed D17
- net D17: now also J118.9 (Pin_9)
- new net: J112.3 (Pin_3), R138.1
- new net: C104.1, C105.1, U118.1 (C1+)
- new net: C104.2, U118.2 (VS+)
- new net: C107.1, U118.4 (C2+)
- new net: C107.2, U118.5 (C2-)
- new net: J112.1 (Pin_1), R140.1
- new net: C105.2, U118.3 (C1-)
- new net: C108.1, U118.6 (VS-)
- new net: J112.5 (Pin_5), R136.1
- new net: J110.1 (Pin_1), R134.1
- new net D13: J115.10 (GPIO15_RXD0), J117.13 (Pin_13), U118.11 (T1IN)
- new net D35: J115.8 (GPIO14_TXD0), J117.5 (Pin_5), U118.12 (R1OUT)
- no-connect marks 0 -> 2
Other:
- note added: "ESP32 DEVKIT"
- moved on the sheet: J119
