File: cad/MoBoControl.kicad_sch (KiCad schematic)
At the start: 112 parts, among them J101 Conn_01x03, J102 Conn_01x03, J103 Conn_01x03, J104 Conn_01x03, J105 Conn_02x04_Odd_Even, J106 Conn_01x03, J107 Conn_01x03, J108 Conn_01x03, J109 power_input, J110 Conn_01x02, J111 USB_A, J112 Conn_02x03_Odd_Even, J113 Conn_01x04, J114 Conn_02x05_Odd_Even, J115 RPi_GPIO, J116 Conn_02x10_Odd_Even, J117 Conn_01x15, J118 Conn_01x15, J119 Conn_02x05_Odd_Even, SW101 SW_Push, SW102 SW_Push, U1 MCP23017, U101 ASSR-1218, U102 ASSR-1218, U103 ASSR-1218, U104 ASSR-1218, U105 ASSR-1218, U106 ASSR-1218, U107 ASSR-1218, U108 ASSR-1218, U109 ASSR-1218, U110 ASSR-1218, U111 ASSR-1218, U112 ASSR-1218, U113 ASSR-1218, U114 ASSR-1218, U115 ASSR-1218, U116 ASSR-1218, U118 MAX232

Commit message: gerbers
Parts:
- R101, R102, R103, R104, R105, R106, R107, R108, R117, R118, R119, R120, R121, R122, R123, R124, R133, R134, R135, R136, R137, R138, R139, R140, R141, R142, R143: value 4.7k -> 220R
- R109, R110, R111, R112, R113, R114, R115, R116, R125, R126, R127, R128, R129, R130: value 10k -> 220R
- renumbered C103 to C102, C102 to C103, J111 to J109, J109 to J110, J116 to J111, J114 to J112, J110 to J113, J117 to J114, J112 to J115, J113 to J116, J118 to J117, J115 to J118, JP103 to JP101, JP101 to JP102, JP102 to JP103
